Commit message: Modificando URDF.

File: urdf/colmena2.gazebo.xacro (robot description, xacro)
@@ -22,13 +22,4 @@
     <material>Gazebo/Black</material>
   </gazebo>
-  <gazebo reference="arm">
-    <material>Gazebo/Gray</material>
-  </gazebo>
-  <gazebo reference="support">
-    <material>Gazebo/Gray</material>
-  </gazebo>
-  <gazebo reference="panel">
-    <material>Gazebo/Blue</material>
-  </gazebo>
   <gazebo>
     <plugin name="skid_steer_drive" filename="libgazebo_ros_diff_drive.so">
@@ -43,6 +34,6 @@
       <wheel_separation>0.22</wheel_separation>
       <wheel_separation>0.22</wheel_separation>
-      <wheel_diameter>0.072</wheel_diameter>
-      <wheel_diameter>0.072</wheel_diameter>
+      <wheel_diameter>0.056</wheel_diameter>
+      <wheel_diameter>0.056</wheel_diameter>
       <max_wheel_torque>1000</max_wheel_torque>
       <max_wheel_acceleration>10.0</max_wheel_acceleration>

File: urdf/colmena2_core.xacro (robot description, xacro)
@@ -5,19 +5,19 @@
   <link name="chassis">
     <inertial>
-      <mass value="2.088534"/>
-      <origin xyz="0 0 0" rpy="0.0 0.0 0.0"/>
-      <inertia
-        ixx="0.004459"
-        ixy="0.0"
-        ixz="0.00009"
-        iyy="0.009908"
-        iyz="0.0"
-        izz="0.01322"
-      />
-    </inertial>
-    <visual>
-      <origin xyz="0 0 0" rpy="0 0 0"/>
-      <geometry>
-        <mesh filename="file://$(find colmena2_description)/meshes/chasis.stl" scale="0.001 0.001 0.001"/>
+      <mass value="2.222"/>
+      <origin xyz="0 0 0" rpy="0.0 0.0 0.0"/>
+      <inertia
+        ixx="0.004757"
+        ixy="0.0"
+        ixz="0.0001595"
+        iyy="0.01069"
+        iyz="0.0"
+        izz="0.01402"
+      />
+    </inertial>
+    <visual>
+      <origin xyz="0 0 0" rpy="0 0 0"/>
+      <geometry>
+        <mesh filename="file://$(find colmena2_description)/meshes/chassis.stl" scale="0.001 0.001 0.001"/>
       </geometry>
       <material name="white"/>
@@ -26,5 +26,32 @@
       <origin xyz="0 0 0" rpy="0 0 0"/>
       <geometry>
-        <mesh filename="file://$(find colmena2_description)/meshes/chasis.stl" scale="0.001 0.001 0.001"/>
+        <mesh filename="file://$(find colmena2_description)/meshes/chassis.stl" scale="0.001 0.001 0.001"/>
+      </geometry>
+    </collision>
+  </link>
+  <link name="left_sprocket">
+    <inertial>
+      <mass value="0.239463"/>
+      <origin xyz="0 0 0" rpy="0.0 0.0 0.0"/>
+      <inertia
+        ixx="0.0000608"
+        ixy="0.0"
+        ixz="0.0"
+        iyy="0.0001084"
+        iyz="0.0"
+        izz="0.0000608"
+      />
+    </inertial>
+    <visual>
+      <origin xyz="0 0 0" rpy="0 0 0"/>
+      <geometry>
+        <mesh filename="file://$(find colmena2_description)/meshes/wheel.stl" scale="0.001 0.001 0.001"/>
+      </geometry>
+      <material name="silver"/>
+    </visual>
+    <collision>
+      <origin xyz="0 0 0" rpy="0 0 0"/>
+      <geometry>
+        <mesh filename="file://$(find colmena2_description)/meshes/wheel.stl" scale="0.001 0.001 0.001"/>
       </geometry>
     </collision>
@@ -32,288 +59,165 @@
   <link name="right_sprocket">
     <inertial>
+      <mass value="0.239463"/>
+      <origin xyz="0 0 0" rpy="0.0 0.0 0.0"/>
+      <inertia
+        ixx="0.0000608"
+        ixy="0.0"
+        ixz="0.0"
+        iyy="0.0001084"
+        iyz="0.0"
+        izz="0.0000608"
+      />
+    </inertial>
+    <visual>
+      <origin xyz="0 0 0" rpy="0 0 0"/>
+      <geometry>
+        <mesh filename="file://$(find colmena2_description)/meshes/wheel.stl" scale="0.001 0.001 0.001"/>
+      </geometry>
+      <material name="silver"/>
+    </visual>
+    <collision>
+      <origin xyz="0 0 0" rpy="0 0 0"/>
+      <geometry>
+        <mesh filename="file://$(find colmena2_description)/meshes/wheel.stl" scale="0.001 0.001 0.001"/>
+      </geometry>
+    </collision>
+  </link>
+  <link name="left_wheel">
+    <inertial>
+      <mass value="0.239463"/>
+      <origin xyz="0 0 0" rpy="0.0 0.0 0.0"/>
+      <inertia
+        ixx="0.0000608"
+        ixy="0.0"
+        ixz="0.0"
+        iyy="0.0001084"
+        iyz="0.0"
+        izz="0.0000608"
+      />
+    </inertial>
+    <visual>
+      <origin xyz="0 0 0" rpy="0 0 0"/>
+      <geometry>
+        <mesh filename="file://$(find colmena2_description)/meshes/wheel.stl" scale="0.001 0.001 0.001"/>
+      </geometry>
+      <material name="silver"/>
+    </visual>
+    <collision>
+      <origin xyz="0 0 0" rpy="0 0 0"/>
+      <geometry>
+        <mesh filename="file://$(find colmena2_description)/meshes/wheel.stl" scale="0.001 0.001 0.001"/>
+      </geometry>
+    </collision>
+  </link>
+  <link name="right_wheel">
+    <inertial>
+      <mass value="0.239463"/>
+      <origin xyz="0 0 0" rpy="0.0 0.0 0.0"/>
+      <inertia
+        ixx="0.0000608"
+        ixy="0.0"
+        ixz="0.0"
+        iyy="0.0001084"
+        iyz="0.0"
+        izz="0.0000608"
+      />
+    </inertial>
+    <visual>
+      <origin xyz="0 0 0" rpy="0 0 0"/>
+      <geometry>
+        <mesh filename="file://$(find colmena2_description)/meshes/wheel.stl" scale="0.001 0.001 0.001"/>
+      </geometry>
+      <material name="silver"/>
+    </visual>
+    <collision>
+      <origin xyz="0 0 0" rpy="0 0 0"/>
+      <geometry>
+        <mesh filename="file://$(find colmena2_description)/meshes/wheel.stl" scale="0.001 0.001 0.001"/>
+      </geometry>
+    </collision>
+  </link>
+  <link name="left_track">
+    <inertial>
       <mass value="0.022541"/>
       <origin xyz="0 0 0" rpy="0.0 0.0 0.0"/>
       <inertia
-        ixx="0.000005"
-        ixy="0.0"
-        ixz="0.0"
-        iyy="0.000009"
-        iyz="0.0"
-        izz="0.000005"
-      />
-    </inertial>
-    <visual>
-      <origin xyz="0 0 0" rpy="0 0 0"/>
-      <geometry>
-        <mesh filename="file://$(find colmena2_description)/meshes/rueda.stl" scale="0.001 0.001 0.001"/>
-      </geometry>
-      <material name="silver"/>
-    </visual>
-    <collision>
-      <origin xyz="0 0 0" rpy="0 0 0"/>
-      <geometry>
-        <mesh filename="file://$(find colmena2_description)/meshes/rueda.stl" scale="0.001 0.001 0.001"/>
-      </geometry>
-    </collision>
-  </link>
-  <link name="left_sprocket">
+        ixx="0.0001033"
+        ixy="0.0"
+        ixz="0.0"
+        iyy="0.0009194"
+        iyz="0.0"
+        izz="0.0008376"
+      />
+    </inertial>
+    <visual>
+      <origin xyz="0 0 0" rpy="0 0 0"/>
+      <geometry>
+        <mesh filename="file://$(find colmena2_description)/meshes/track.stl" scale="0.001 0.001 0.001"/>
+      </geometry>
+      <material name="black"/>
+    </visual>
+  </link>
+  <link name="right_track">
     <inertial>
       <mass value="0.022541"/>
       <origin xyz="0 0 0" rpy="0.0 0.0 0.0"/>
       <inertia
-        ixx="0.000005"
-        ixy="0.0"
-        ixz="0.0"
-        iyy="0.000009"
-        iyz="0.0"
-        izz="0.000005"
-      />
-    </inertial>
-    <visual>
-      <origin xyz="0 0 0" rpy="0 0 0"/>
-      <geometry>
-        <mesh filename="file://$(find colmena2_description)/meshes/rueda.stl" scale="0.001 0.001 0.001"/>
-      </geometry>
-      <material name="silver"/>
-    </visual>
-    <collision>
-      <origin xyz="0 0 0" rpy="0 0 0"/>
-      <geometry>
-        <mesh filename="file://$(find colmena2_description)/meshes/rueda.stl" scale="0.001 0.001 0.001"/>
-      </geometry>
-    </collision>
-  </link>
-  <link name="right_wheel">
-    <inertial>
-      <mass value="0.022541"/>
-      <origin xyz="0 0 0" rpy="0.0 0.0 0.0"/>
-      <inertia
-        ixx="0.000005"
-        ixy="0.0"
-        ixz="0.0"
-        iyy="0.000009"
-        iyz="0.0"
-        izz="0.000005"
-      />
-    </inertial>
-    <visual>
-      <origin xyz="0 0 0" rpy="0 0 0"/>
-      <geometry>
-        <mesh filename="file://$(find colmena2_description)/meshes/rueda.stl" scale="0.001 0.001 0.001"/>
-      </geometry>
-      <material name="silver"/>
-    </visual>
-    <collision>
-      <origin xyz="0 0 0" rpy="0 0 0"/>
-      <geometry>
-        <mesh filename="file://$(find colmena2_description)/meshes/rueda.stl" scale="0.001 0.001 0.001"/>
-      </geometry>
-    </collision>
-  </link>
-  <link name="left_wheel">
-    <inertial>
-      <mass value="0.022541"/>
-      <origin xyz="0 0 0" rpy="0.0 0.0 0.0"/>
-      <inertia
-        ixx="0.000005"
-        ixy="0.0"
-        ixz="0.0"
-        iyy="0.000009"
-        iyz="0.0"
-        izz="0.000005"
-      />
-    </inertial>
-    <visual>
-      <origin xyz="0 0 0" rpy="0 0 0"/>
-      <geometry>
-        <mesh filename="file://$(find colmena2_description)/meshes/rueda.stl" scale="0.001 0.001 0.001"/>
-      </geometry>
-      <material name="silver"/>
-    </visual>
-    <collision>
-      <origin xyz="0 0 0" rpy="0 0 0"/>
-      <geometry>
-        <mesh filename="file://$(find colmena2_description)/meshes/rueda.stl" scale="0.001 0.001 0.001"/>
-      </geometry>
-    </collision>
-  </link>
-  <link name="right_track">
-    <inertial>
-      <mass value="0.022541"/>
-      <origin xyz="0 0 0" rpy="0.0 0.0 0.0"/>
-      <inertia
-        ixx="0.000064"
-        ixy="0.0"
-        ixz="0.0"
-        iyy="0.000599"
-        iyz="0.0"
-        izz="0.000541"
-      />
-    </inertial>
-    <visual>
-      <origin xyz="0 0 0" rpy="0 0 0"/>
-      <geometry>
-        <mesh filename="file://$(find colmena2_description)/meshes/oruga.stl" scale="0.001 0.001 0.001"/>
+        ixx="0.0001033"
+        ixy="0.0"
+        ixz="0.0"
+        iyy="0.0009194"
+        iyz="0.0"
+        izz="0.0008376"
+      />
+    </inertial>
+    <visual>
+      <origin xyz="0 0 0" rpy="0 0 0"/>
+      <geometry>
+        <mesh filename="file://$(find colmena2_description)/meshes/track.stl" scale="0.001 0.001 0.001"/>
       </geometry>
       <material name="black"/>
     </visual>
-  </link>
-  <link name="left_track">
-    <inertial>
-      <mass value="0.022541"/>
-      <origin xyz="0 0 0" rpy="0.0 0.0 0.0"/>
-      <inertia
-        ixx="0.000064"
-        ixy="0.0"
-        ixz="0.0"
-        iyy="0.000599"
-        iyz="0.0"
-        izz="0.000541"
-      />
-    </inertial>
-    <visual>
-      <origin xyz="0 0 0" rpy="0 0 0"/>
-      <geometry>
-        <mesh filename="file://$(find colmena2_description)/meshes/oruga.stl" scale="0.001 0.001 0.001"/>
-      </geometry>
-      <material name="black"/>
-    </visual>
-  </link>
-  <link name="arm">
-    <inertial>
-      <mass value="0.379695"/>
-      <origin xyz="0 0 0" rpy="0.0 0.0 0.0"/>
-      <inertia
-        ixx="0.000271"
-        ixy="0.0"
-        ixz="0.000359"
-        iyy="0.002343"
-        iyz="0.0"
-        izz="0.002193"
-      />
-    </inertial>
-    <visual>
-      <origin xyz="0 0 0" rpy="0 0 0"/>
-      <geometry>
-        <mesh filename="file://$(find colmena2_description)/meshes/brazo.stl" scale="0.001 0.001 0.001"/>
-      </geometry>
-      <material name="silver"/>
-    </visual>
-    <collision>
-      <origin xyz="0 0 0" rpy="0 0 0"/>
-      <geometry>
-        <mesh filename="file://$(find colmena2_description)/meshes/brazo.stl" scale="0.001 0.001 0.001"/>
-      </geometry>
-    </collision>
-  </link>
-  <link name="support">
-    <inertial>
-      <mass value="0.279375"/>
-      <origin xyz="0 0 0" rpy="0.0 0.0 0.0"/>
-      <inertia
-        ixx="0.000571"
-        ixy="0.0"
-        ixz="-0.00063"
-        iyy="0.000615"
-        iyz="0.0"
-        izz="0.000074"
-      />
-    </inertial>
-    <visual>
-      <origin xyz="0 0 0" rpy="0 0 0"/>
-      <geometry>
-        <mesh filename="file://$(find colmena2_description)/meshes/soporte.stl" scale="0.001 0.001 0.001"/>
-      </geometry>
-      <material name="silver"/>
-    </visual>
-    <collision>
-      <origin xyz="0 0 0" rpy="0 0 0"/>
-      <geometry>
-        <mesh filename="file://$(find colmena2_description)/meshes/soporte.stl" scale="0.001 0.001 0.001"/>
-      </geometry>
-    </collision>
-  </link>
-  <link name="panel">
-    <inertial>
-      <mass value="0.167424"/>
-      <origin xyz="0 0 0" rpy="0.0 0.0 0.0"/>
-      <inertia
-        ixx="0.000265"
-        ixy="0.0"
-        ixz="-0.000137"
-        iyy="0.000357"
-        iyz="0.0"
-        izz="0.000494"
-      />
-    </inertial>
-    <visual>
-      <origin xyz="0 0 0" rpy="0 0 0"/>
-      <geometry>
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
Commit message: Añadiendo archivos STL.

File: urdf/colmena2.gazebo.xacro (robot description, xacro)
@@ -21,4 +21,13 @@
   <gazebo reference="left_track">
     <material>Gazebo/Black</material>
+  </gazebo>
+  <gazebo reference="arm">
+    <material>Gazebo/Gray</material>
+  </gazebo>
+  <gazebo reference="support">
+    <material>Gazebo/Gray</material>
+  </gazebo>
+  <gazebo reference="panel">
+    <material>Gazebo/Blue</material>
   </gazebo>
   <gazebo>

File: urdf/colmena2_core.xacro (robot description, xacro)
@@ -5,13 +5,13 @@
   <link name="chassis">
     <inertial>
-      <mass value="2.222"/>
-      <origin xyz="0 0 0" rpy="0.0 0.0 0.0"/>
-      <inertia
-        ixx="0.004757"
-        ixy="0.0"
-        ixz="0.0001595"
-        iyy="0.01069"
-        iyz="0.0"
-        izz="0.01402"
+      <mass value="2.131"/>
+      <origin xyz="0 0 0" rpy="0.0 0.0 0.0"/>
+      <inertia
+        ixx="0.004055"
+        ixy="0.0"
+        ixz="0.0001573"
+        iyy="0.01032"
+        iyz="0.0"
+        izz="0.01298"
       />
     </inertial>
@@ -179,14 +179,95 @@
       <material name="black"/>
     </visual>
+  </link>
+  <link name="arm">
+    <inertial>
+      <mass value="0.369"/>
+      <origin xyz="0 0 0" rpy="0.0 0.0 0.0"/>
+      <inertia
+        ixx="0.0001981"
+        ixy="0.0"
+        ixz="-0.0000834"
+        iyy="0.002241"
+        iyz="0.0"
+        izz="0.002158"
+      />
+    </inertial>
+    <visual>
+      <origin xyz="0 0 0" rpy="0 0 0"/>
+      <geometry>
+        <mesh filename="file://$(find colmena2_description)/meshes/arm.stl" scale="0.001 0.001 0.001"/>
+      </geometry>
+      <material name="silver"/>
+    </visual>
+    <collision>
+      <origin xyz="0 0 0" rpy="0 0 0"/>
+      <geometry>
+        <mesh filename="file://$(find colmena2_description)/meshes/arm.stl" scale="0.001 0.001 0.001"/>
+      </geometry>
+    </collision>
+  </link>
+  <link name="support">
+    <inertial>
+      <mass value="0.280"/>
+      <origin xyz="0 0 0" rpy="0.0 0.0 0.0"/>
+      <inertia
+        ixx="0.0005618"
+        ixy="0.0"
+        ixz="-0.0001057"
+        iyy="0.0006207"
+        iyz="0.0"
+        izz="0.0000886"
+      />
+    </inertial>
+    <visual>
+      <origin xyz="0 0 0" rpy="0 0 0"/>
+      <geometry>
+        <mesh filename="file://$(find colmena2_description)/meshes/support.stl" scale="0.001 0.001 0.001"/>
+      </geometry>
+      <material name="silver"/>
+    </visual>
+    <collision>
+      <origin xyz="0 0 0" rpy="0 0 0"/>
+      <geometry>
+        <mesh filename="file://$(find colmena2_description)/meshes/support.stl" scale="0.001 0.001 0.001"/>
+      </geometry>
+    </collision>
+  </link>
+  <link name="panel">
+    <inertial>
+      <mass value="0.167"/>
+      <origin xyz="0 0 0" rpy="0.0 0.0 0.0"/>
+      <inertia
+        ixx="0.0002904"
+        ixy="0.0"
+        ixz="0.0001546"
+        iyy="0.0003574"
+        iyz="0.0"
+        izz="0.0004688"
+      />
+    </inertial>
+    <visual>
+      <origin xyz="0 0 0" rpy="0 0 0"/>
+      <geometry>
+        <mesh filename="file://$(find colmena2_description)/meshes/panel.stl" scale="0.001 0.001 0.001"/>
+      </geometry>
+      <material name="blue"/>
+    </visual>
+    <collision>
+      <origin xyz="0 0 0" rpy="0 0 0"/>
+      <geometry>
+        <mesh filename="file://$(find colmena2_description)/meshes/panel.stl" scale="0.001 0.001 0.001"/>
+      </geometry>
+    </collision>
   </link>
   <joint name="ch_to_bl_joint" type="fixed">
     <parent link="base_link"/>
     <child link="chassis"/>
-    <origin xyz="-0.002361 -0.000004 0.009671"/>
+    <origin xyz="-0.002463 -0.000004 0.010086"/>
   </joint>
   <joint name="ls_to_ch_joint" type="continuous">
     <parent link="chassis"/>
     <child link="left_sprocket"/>
-    <origin xyz="-0.097639 0.110004 -0.009671"/>
+    <origin xyz="-0.097537 0.100004 -0.010086"/>
     <axis xyz="0 1 0"/>
   </joint>
@@ -194,5 +275,5 @@
     <parent link="chassis"/>
     <child link="right_sprocket"/>
-    <origin xyz="-0.097639 -0.109996 -0.009671"/>
+    <origin xyz="-0.097537 -0.099996 -0.010086"/>
     <axis xyz="0 1 0"/>
   </joint>
@@ -200,5 +281,5 @@
     <parent link="chassis"/>
     <child link="left_wheel"/>
-    <origin xyz="0.102361 0.110004 -0.009671"/>
+    <origin xyz="0.102463 0.100004 -0.010086"/>
     <axis xyz="0 1 0"/>
     <mimic joint="ls_to_ch_joint" multiplier="1" offset="0"/>
@@ -207,5 +288,5 @@
     <parent link="chassis"/>
     <child link="right_wheel"/>
-    <origin xyz="0.102361 -0.109996 -0.009671"/>
+    <origin xyz="0.102463 -0.099996 -0.010086"/>
     <axis xyz="0 1 0"/>
     <mimic joint="rs_to_ch_joint" multiplier="1" offset="0"/>
@@ -214,10 +295,25 @@
     <parent link="chassis"/>
     <child link="left_track"/>
-    <origin xyz="0.002356 0.110004 -0.009671"/>
+    <origin xyz="0.002458 0.100004 -0.010086"/>
   </joint>
   <joint name="rt_to_ch_joint" type="fixed">
     <parent link="chassis"/>
     <child link="right_track"/>
-    <origin xyz="0.002356 -0.109996 -0.009671"/>
+    <origin xyz="0.002458 -0.099996 -0.010086"/>
+  </joint>
+  <joint name="arm_to_ch_joint" type="fixed">
+    <parent link="chassis"/>
+    <child link="arm"/>
+    <origin xyz="0.243999 0.0 0.071118"/>
+  </joint>
+  <joint name="sp_to_ch_joint" type="fixed">
+    <parent link="chassis"/>
+    <child link="support"/>
+    <origin xyz="-0.070318 0.0 0.112644"/>
+  </joint>
+  <joint name="pn_to_ch_joint" type="fixed">
+    <parent link="chassis"/>
+    <child link="panel"/>
+    <origin xyz="-0.035091 0.000003 0.196115" rpy="0.0 ${pi/6} 0.0"/>
   </joint>
 </robot>
