Commit message: Modificando archivos STL.

File: urdf/colmena2.gazebo.xacro (robot description, xacro)
@@ -5,14 +5,14 @@
   </gazebo>
   <gazebo reference="right_sprocket">
-    <material>Gazebo/Gray</material>
+    <material>Gazebo/Black</material>
   </gazebo>
   <gazebo reference="right_wheel">
-    <material>Gazebo/Gray</material>
+    <material>Gazebo/Black</material>
   </gazebo>
   <gazebo reference="left_sprocket">
-    <material>Gazebo/Gray</material>
+    <material>Gazebo/Black</material>
   </gazebo>
   <gazebo reference="left_wheel">
-    <material>Gazebo/Gray</material>
+    <material>Gazebo/Black</material>
   </gazebo>
   <gazebo reference="right_track">
@@ -21,13 +21,4 @@
   <gazebo reference="left_track">
     <material>Gazebo/Black</material>
-  </gazebo>
-  <gazebo reference="arm">
-    <material>Gazebo/Gray</material>
-  </gazebo>
-  <gazebo reference="support">
-    <material>Gazebo/Gray</material>
-  </gazebo>
-  <gazebo reference="panel">
-    <material>Gazebo/Blue</material>
   </gazebo>
   <gazebo>
@@ -41,8 +32,8 @@
       <left_joint>ls_to_ch_joint</left_joint>
       <right_joint>rs_to_ch_joint</right_joint>
-      <wheel_separation>0.22</wheel_separation>
-      <wheel_separation>0.22</wheel_separation>
-      <wheel_diameter>0.056</wheel_diameter>
-      <wheel_diameter>0.056</wheel_diameter>
+      <wheel_separation>0.099</wheel_separation>
+      <wheel_separation>0.099</wheel_separation>
+      <wheel_diameter>0.047</wheel_diameter>
+      <wheel_diameter>0.047</wheel_diameter>
       <max_wheel_torque>1000</max_wheel_torque>
       <max_wheel_acceleration>10.0</max_wheel_acceleration>

File: urdf/colmena2_core.xacro (robot description, xacro)
@@ -5,13 +5,13 @@
   <link name="chassis">
     <inertial>
-      <mass value="2.131"/>
-      <origin xyz="0 0 0" rpy="0.0 0.0 0.0"/>
-      <inertia
-        ixx="0.004055"
-        ixy="0.0"
-        ixz="0.0001573"
-        iyy="0.01032"
-        iyz="0.0"
-        izz="0.01298"
+      <mass value="0.298408"/>
+      <origin xyz="0 0 0" rpy="0.0 0.0 0.0"/>
+      <inertia
+        ixx="0.0003667"
+        ixy="-0.0000122"
+        ixz="0.0000112"
+        iyy="0.0005734"
+        iyz="-0.0000046"
+        izz="0.00006682"
       />
     </inertial>
@@ -32,21 +32,21 @@
   <link name="left_sprocket">
     <inertial>
-      <mass value="0.239463"/>
-      <origin xyz="0 0 0" rpy="0.0 0.0 0.0"/>
-      <inertia
-        ixx="0.0000608"
-        ixy="0.0"
-        ixz="0.0"
-        iyy="0.0001084"
-        iyz="0.0"
-        izz="0.0000608"
-      />
-    </inertial>
-    <visual>
-      <origin xyz="0 0 0" rpy="0 0 0"/>
-      <geometry>
-        <mesh filename="file://$(find colmena2_description)/meshes/wheel.stl" scale="0.001 0.001 0.001"/>
-      </geometry>
-      <material name="silver"/>
+      <mass value="0.051528"/>
+      <origin xyz="0 0 0" rpy="0.0 0.0 0.0"/>
+      <inertia
+        ixx="0.0000098"
+        ixy="0.0"
+        ixz="0.0"
+        iyy="0.0000142"
+        iyz="0.0"
+        izz="0.0000098"
+      />
+    </inertial>
+    <visual>
+      <origin xyz="0 0 0" rpy="0 0 0"/>
+      <geometry>
+        <mesh filename="file://$(find colmena2_description)/meshes/wheel.stl" scale="0.001 0.001 0.001"/>
+      </geometry>
+      <material name="black"/>
     </visual>
     <collision>
@@ -59,21 +59,21 @@
   <link name="right_sprocket">
     <inertial>
-      <mass value="0.239463"/>
-      <origin xyz="0 0 0" rpy="0.0 0.0 0.0"/>
-      <inertia
-        ixx="0.0000608"
-        ixy="0.0"
-        ixz="0.0"
-        iyy="0.0001084"
-        iyz="0.0"
-        izz="0.0000608"
-      />
-    </inertial>
-    <visual>
-      <origin xyz="0 0 0" rpy="0 0 0"/>
-      <geometry>
-        <mesh filename="file://$(find colmena2_description)/meshes/wheel.stl" scale="0.001 0.001 0.001"/>
-      </geometry>
-      <material name="silver"/>
+      <mass value="0.051528"/>
+      <origin xyz="0 0 0" rpy="0.0 0.0 0.0"/>
+      <inertia
+        ixx="0.0000098"
+        ixy="0.0"
+        ixz="0.0"
+        iyy="0.0000142"
+        iyz="0.0"
+        izz="0.0000098"
+      />
+    </inertial>
+    <visual>
+      <origin xyz="0 0 0" rpy="0 0 0"/>
+      <geometry>
+        <mesh filename="file://$(find colmena2_description)/meshes/wheel.stl" scale="0.001 0.001 0.001"/>
+      </geometry>
+      <material name="black"/>
     </visual>
     <collision>
@@ -86,21 +86,21 @@
   <link name="left_wheel">
     <inertial>
-      <mass value="0.239463"/>
-      <origin xyz="0 0 0" rpy="0.0 0.0 0.0"/>
-      <inertia
-        ixx="0.0000608"
-        ixy="0.0"
-        ixz="0.0"
-        iyy="0.0001084"
-        iyz="0.0"
-        izz="0.0000608"
-      />
-    </inertial>
-    <visual>
-      <origin xyz="0 0 0" rpy="0 0 0"/>
-      <geometry>
-        <mesh filename="file://$(find colmena2_description)/meshes/wheel.stl" scale="0.001 0.001 0.001"/>
-      </geometry>
-      <material name="silver"/>
+      <mass value="0.051528"/>
+      <origin xyz="0 0 0" rpy="0.0 0.0 0.0"/>
+      <inertia
+        ixx="0.0000098"
+        ixy="0.0"
+        ixz="0.0"
+        iyy="0.0000142"
+        iyz="0.0"
+        izz="0.0000098"
+      />
+    </inertial>
+    <visual>
+      <origin xyz="0 0 0" rpy="0 0 0"/>
+      <geometry>
+        <mesh filename="file://$(find colmena2_description)/meshes/wheel.stl" scale="0.001 0.001 0.001"/>
+      </geometry>
+      <material name="black"/>
     </visual>
     <collision>
@@ -113,21 +113,21 @@
   <link name="right_wheel">
     <inertial>
-      <mass value="0.239463"/>
-      <origin xyz="0 0 0" rpy="0.0 0.0 0.0"/>
-      <inertia
-        ixx="0.0000608"
-        ixy="0.0"
-        ixz="0.0"
-        iyy="0.0001084"
-        iyz="0.0"
-        izz="0.0000608"
-      />
-    </inertial>
-    <visual>
-      <origin xyz="0 0 0" rpy="0 0 0"/>
-      <geometry>
-        <mesh filename="file://$(find colmena2_description)/meshes/wheel.stl" scale="0.001 0.001 0.001"/>
-      </geometry>
-      <material name="silver"/>
+      <mass value="0.051528"/>
+      <origin xyz="0 0 0" rpy="0.0 0.0 0.0"/>
+      <inertia
+        ixx="0.0000098"
+        ixy="0.0"
+        ixz="0.0"
+        iyy="0.0000142"
+        iyz="0.0"
+        izz="0.0000098"
+      />
+    </inertial>
+    <visual>
+      <origin xyz="0 0 0" rpy="0 0 0"/>
+      <geometry>
+        <mesh filename="file://$(find colmena2_description)/meshes/wheel.stl" scale="0.001 0.001 0.001"/>
+      </geometry>
+      <material name="black"/>
     </visual>
     <collision>
@@ -140,13 +140,13 @@
   <link name="left_track">
     <inertial>
-      <mass value="0.022541"/>
-      <origin xyz="0 0 0" rpy="0.0 0.0 0.0"/>
-      <inertia
-        ixx="0.0001033"
-        ixy="0.0"
-        ixz="0.0"
-        iyy="0.0009194"
-        iyz="0.0"
-        izz="0.0008376"
+      <mass value="0.049475"/>
+      <origin xyz="0 0 0" rpy="0.0 0.0 0.0"/>
+      <inertia
+        ixx="0.0000208"
+        ixy="0.0"
+        ixz="0.0"
+        iyy="0.0001660"
+        iyz="0.0"
+        izz="0.0001504"
       />
     </inertial>
@@ -161,13 +161,13 @@
   <link name="right_track">
     <inertial>
-      <mass value="0.022541"/>
-      <origin xyz="0 0 0" rpy="0.0 0.0 0.0"/>
-      <inertia
-        ixx="0.0001033"
-        ixy="0.0"
-        ixz="0.0"
-        iyy="0.0009194"
-        iyz="0.0"
-        izz="0.0008376"
+      <mass value="0.049475"/>
+      <origin xyz="0 0 0" rpy="0.0 0.0 0.0"/>
+      <inertia
+        ixx="0.0000208"
+        ixy="0.0"
+        ixz="0.0"
+        iyy="0.0001660"
+        iyz="0.0"
+        izz="0.0001504"
       />
     </inertial>
@@ -179,95 +179,14 @@
       <material name="black"/>
     </visual>
-  </link>
-  <link name="arm">
-    <inertial>
-      <mass value="0.369"/>
-      <origin xyz="0 0 0" rpy="0.0 0.0 0.0"/>
-      <inertia
-        ixx="0.0001981"
-        ixy="0.0"
-        ixz="-0.0000834"
-        iyy="0.002241"
-        iyz="0.0"
-        izz="0.002158"
-      />
-    </inertial>
-    <visual>
-      <origin xyz="0 0 0" rpy="0 0 0"/>
-      <geometry>
-        <mesh filename="file://$(find colmena2_description)/meshes/arm.stl" scale="0.001 0.001 0.001"/>
-      </geometry>
-      <material name="silver"/>
-    </visual>
-    <collision>
-      <origin xyz="0 0 0" rpy="0 0 0"/>
-      <geometry>
-        <mesh filename="file://$(find colmena2_description)/meshes/arm.stl" scale="0.001 0.001 0.001"/>
-      </geometry>
-    </collision>
-  </link>
-  <link name="support">
-    <inertial>
-      <mass value="0.280"/>
-      <origin xyz="0 0 0" rpy="0.0 0.0 0.0"/>
-      <inertia
-        ixx="0.0005618"
-        ixy="0.0"
-        ixz="-0.0001057"
-        iyy="0.0006207"
-        iyz="0.0"
-        izz="0.0000886"
-      />
-    </inertial>
-    <visual>
-      <origin xyz="0 0 0" rpy="0 0 0"/>
-      <geometry>
-        <mesh filename="file://$(find colmena2_description)/meshes/support.stl" scale="0.001 0.001 0.001"/>
-      </geometry>
-      <material name="silver"/>
-    </visual>
-    <collision>
-      <origin xyz="0 0 0" rpy="0 0 0"/>
-      <geometry>
-        <mesh filename="file://$(find colmena2_description)/meshes/support.stl" scale="0.001 0.001 0.001"/>
-      </geometry>
-    </collision>
-  </link>
-  <link name="panel">
-    <inertial>
-      <mass value="0.167"/>
-      <origin xyz="0 0 0" rpy="0.0 0.0 0.0"/>
-      <inertia
-        ixx="0.0002904"
-        ixy="0.0"
-        ixz="0.0001546"
-        iyy="0.0003574"
-        iyz="0.0"
-        izz="0.0004688"
-      />
-    </inertial>
-    <visual>
-      <origin xyz="0 0 0" rpy="0 0 0"/>
-      <geometry>
-        <mesh filename="file://$(find colmena2_description)/meshes/panel.stl" scale="0.001 0.001 0.001"/>
-      </geometry>
-      <material name="blue"/>
-    </visual>
-    <collision>
-      <origin xyz="0 0 0" rpy="0 0 0"/>
-      <geometry>
-        <mesh filename="file://$(find colmena2_description)/meshes/panel.stl" scale="0.001 0.001 0.001"/>
-      </geometry>
-    </collision>
   </link>
   <joint name="ch_to_bl_joint" type="fixed">
     <parent link="base_link"/>
     <child link="chassis"/>
-    <origin xyz="-0.002463 -0.000004 0.010086"/>
+    <origin xyz="-0.007614 0.000962 0.01313"/>
   </joint>
   <joint name="ls_to_ch_joint" type="continuous">
     <parent link="chassis"/>
     <child link="left_sprocket"/>
-    <origin xyz="-0.097537 0.100004 -0.010086"/>
+    <origin xyz="-0.056886 0.048538 -0.01313"/>
     <axis xyz="0 1 0"/>
   </joint>
@@ -275,5 +194,5 @@
     <parent link="chassis"/>
     <child link="right_sprocket"/>
-    <origin xyz="-0.097537 -0.099996 -0.010086"/>
+    <origin xyz="-0.056886 -0.050462 -0.01313"/>
     <axis xyz="0 1 0"/>
   </joint>
@@ -281,5 +200,5 @@
     <parent link="chassis"/>
     <child link="left_wheel"/>
-    <origin xyz="0.102463 0.100004 -0.010086"/>
+    <origin xyz="0.072114 0.048538 -0.01313"/>
     <axis xyz="0 1 0"/>
     <mimic joint="ls_to_ch_joint" multiplier="1" offset="0"/>
@@ -288,5 +207,5 @@
     <parent link="chassis"/>
     <child link="right_wheel"/>
-    <origin xyz="0.102463 -0.099996 -0.010086"/>
+    <origin xyz="0.072114 -0.050462 -0.01313"/>
     <axis xyz="0 1 0"/>
     <mimic joint="rs_to_ch_joint" multiplier="1" offset="0"/>
@@ -295,25 +214,10 @@
     <parent link="chassis"/>
     <child link="left_track"/>
-    <origin xyz="0.002458 0.100004 -0.010086"/>
+    <origin xyz="0.007614 0.048538 -0.01313"/>
   </joint>
   <joint name="rt_to_ch_joint" type="fixed">
     <parent link="chassis"/>
     <child link="right_track"/>
-    <origin xyz="0.002458 -0.099996 -0.010086"/>
-  </joint>
-  <joint name="arm_to_ch_joint" type="fixed">
-    <parent link="chassis"/>
-    <child link="arm"/>
-    <origin xyz="0.243999 0.0 0.071118"/>
-  </joint>
-  <joint name="sp_to_ch_joint" type="fixed">
-    <parent link="chassis"/>
-    <child link="support"/>
-    <origin xyz="-0.070318 0.0 0.112644"/>
-  </joint>
-  <joint name="pn_to_ch_joint" type="fixed">
-    <parent link="chassis"/>
-    <child link="panel"/>
-    <origin xyz="-0.035091 0.000003 0.196115" rpy="0.0 ${pi/6} 0.0"/>
+    <origin xyz="0.007614 -0.050462 -0.01313"/>
   </joint>
 </robot>

File: urdf/materials.xacro (robot description, xacro)
@@ -4,15 +4,6 @@
     <color rgba="0.200 0.200 0.200 1.000"/> <!-- Negro -->
   </material>
-  <material name="silver">
-    <color rgba="0.600 0.600 0.600 1.000"/> <!-- Plata -->
-  </material>
-  <material name="red">
-    <color rgba="1.000 0.000 0.000 1.000"/> <!-- Rojo -->
-  </material>
   <material name="white">
     <color rgba="1.000 1.000 1.000 1.000"/> <!-- Blanco -->
   </material>
-  <material name="blue">
-    <color rgba="0.000 0.300 1.000 1.000"/> <!-- Azul -->
-  </material>
 </robot>
